File: PCBs/Mirto Pico/Mirtle_Pico_Hotec_drv8833_pi.brd (EAGLE design)
At the start: 56 x 76 mm, 40 parts, among them SW1 OS102011MA1Q, U1 RASPBERRY_PICOTH

Commit message: updated build doc updated bumper dxf
Parts:
- removed I2C: (no value), SparkFun-Connectors:1X04
- removed RN2: (no value), resistor-sil:SIL5
- added 3V3ZENER: (no value), diode:ZDIO-5
- added R1, R4, R5: 4.7k, resistor:0204/5
Connections:
- removed net SCL0: AUX_5V.2, I2C.2, PI.4, RN2.4, U1.22
- removed net SDA0: AUX_5V.1, I2C.1, PI.5, RN2.5, U1.21
- new net RX0: 3V3ZENER.A, PI.4, R1.2, U1.22
- new net RX5V: AUX_5V.2, R1.1
- new net TX0: AUX_5V.1, PI.5, U1.21
- net GND: now also 3V3ZENER.C; no longer I2C.4
- net SCL1: now also R5.1; no longer RN2.2
- net SDA1: now also R4.1; no longer RN2.3
- net VCC: now also R4.2, R5.2; no longer I2C.3, RN2.1
Routing:
- net TX0: track 0.00 -> 45.7 mm
- net RX0: track 0.00 -> 45.1 mm
- net SCL0: track 45.1 -> 0.00 mm
- net SDA0: track 43.4 -> 0.00 mm
- net GND: track 332.8 -> 353.0 mm
- net RX5V: track 0.00 -> 9.13 mm
- net SERVO: track 25.8 -> 19.1 mm
- net VCC: track 135.4 -> 130.0 mm
- net SCL1: track 23.5 -> 19.7 mm
- net SDA1: track 20.8 -> 17.4 mm
Other:
- board text added: "5V"
- board text added: "5V Serial"
- board text added: "Rx"
- board text added: "Tx"
- board text removed: "SDA SCL 3.3 Gnd"
