File: PCBs/Mirto Pico/Mirtle_Pico_Hotec_drv8833_pi.sch (EAGLE design)
At the start: 40 parts, among them SW1 OS102011MA1Q, U1 RASPBERRY_PICOTH

Commit message: updated build doc updated bumper dxf
Parts:
- removed I2C: (no value), SparkFun-Connectors:CONN_04
- removed RN2: (no value), resistor-sil:G04R
- added 3V3ZENER: (no value), diode:ZENER-DIODEZD-5
- added R1, R4, R5: 4.7k, resistor:R-EU_0204/5
Connections:
- removed net SCL0: AUX_5V.2, I2C.2, PI.4, RN2.4, U1.GP17
- removed net SDA0: AUX_5V.1, I2C.1, PI.5, RN2.5, U1.GP16
- new net RX0: 3V3ZENER.A, PI.4, R1.2, U1.GP17
- new net RX5V: AUX_5V.2, R1.1
- new net TX0: AUX_5V.1, PI.5, U1.GP16
- net GND: now also 3V3ZENER.C; no longer I2C.4
- net SCL1: now also R5.1; no longer RN2.2
- net SDA1: now also R4.1; no longer RN2.3
- net VCC: now also R4.2, R5.2; no longer I2C.3, RN2.1
Other:
- note added: "3.3Volt I2C on Bus 1"
- note added: "5 Volt I2C on Bus 0 or Serial"
- moved on the sheet: AUX_5V
